File: 42's_bootcamp/42's_bootcamp.kicad_pcb (KiCad board)
At the start: 2 copper layers, 59 x 41.5 mm, 17 parts, among them J3 FTDI, SW1 SW_PUSH, U1 ATmega328P-A

Commit message: finished
Parts:
- moved C4 47.7 mm to (140.0, 60.5)
- moved SW1 43.4 mm to (141.0, 65.5), turned to -90 degrees
- moved R3 42.5 mm to (140.0, 62.0)
- moved D1 31.8 mm to (160.5, 63.5), turned to -90 degrees
- moved R1 29.0 mm to (160.5, 60.0), turned to -90 degrees
- moved C7 24.5 mm to (144.0, 60.0), turned to 90 degrees
- moved D2 24.2 mm to (145.5, 60.0), turned to -90 degrees
- moved R2 23.9 mm to (144.5, 62.5), turned to 180 degrees
- moved C6 21.0 mm to (142.5, 60.0), turned to 90 degrees
- moved C3 15.3 mm to (157.0, 61.0), turned to 135 degrees
- moved J1 9.51 mm to (150.7, 77.2)
- moved Y1 8.63 mm to (142.5, 72.2), turned to 180 degrees
- moved C2 6.95 mm to (146.5, 70.0), turned to 180 degrees
- moved J2 6.67 mm to (149.2, 55.3)
- moved C1 4.92 mm to (146.5, 73.0), turned to 180 degrees
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Routing:
- net GND: track 0.00 -> 81.4 mm, vias 0 -> 3
- net RAW: track 0.00 -> 66.4 mm
- net DTR: track 0.00 -> 62.3 mm
- net RXI: track 0.00 -> 30.5 mm
- net D4: track 0.00 -> 24.9 mm
- net D3: track 0.00 -> 23.0 mm
- net TXO: track 0.00 -> 22.6 mm
- net D2: track 0.00 -> 22.2 mm
- net D10: track 0.00 -> 19.1 mm
- net MOSI: track 0.00 -> 17.8 mm
- net SCK: track 0.00 -> 16.7 mm
- net MISO: track 0.00 -> 16.2 mm
- net D9: track 0.00 -> 10.7 mm
- net D8: track 0.00 -> 9.13 mm
- net A3: track 0.00 -> 8.35 mm
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- removed copper zone on B.Cu, net GND
Other:
- board size 59 x 41.5 mm -> 31.5 x 24.9 mm
