File: 42's_bootcamp/42's_bootcamp.kicad_sch (KiCad schematic)
At the start: 17 parts, among them J3 FTDI, SW1 SW_PUSH, U1 ATmega328P-A

Commit message: time connected
Parts:
- C1, C2, C3, C4, C6, C7: footprint (none) -> pkorsako_footprint:C_0603
- D1, D2: footprint (none) -> pkorsako_footprint:Led_0603
- J1, J2: footprint (none) -> pkorsako_footprint:PinHeader_1x12_P2.54mm
- J3: footprint (none) -> pkorsako_footprint:PinHeader_1x06_P2.54mm
- R1, R2, R3: footprint (none) -> pkorsako_footprint:R_0603
- SW1: footprint (none) -> pkorsako_footprint:SW_SPST_B3U-1000P
- U1: footprint (none) -> pkorsako_footprint:TQFP-32_7x7_Pitch0.8mm
- Y1: footprint (none) -> pkorsako_footprint:Crystal_SMD_3225
Changed lines of the file:
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@@
 	)
 	(junction
-		(at 27.94 34.29)
+		(at 31.75 92.71)
 		(diameter 0)
 		(color 0 0 0 0)
 	)
 	(junction
-		(at 31.75 92.71)
+		(at 27.94 34.29)
 		(diameter 0)
 		(color 0 0 0 0)
@@
 			)
 		)
-		(property "Footprint" ""
+		(property "Footprint" "pkorsako_footprint:C_0603"
 			(at 109.22 130.81 0)
 			(hide yes)
@@
 			)
 		)
-		(property "Footprint" ""
+		(property "Footprint" "pkorsako_footprint:C_0603"
 			(at 109.22 113.03 0)
 			(hide yes)
@@
 			)
 		)
-		(property "Footprint" ""
+		(property "Footprint" "pkorsako_footprint:PinHeader_1x12_P2.54mm"
 			(at 184.15 140.97 0)
 			(hide yes)
@@
 			)
 		)
-		(property "Footprint" ""
+		(property "Footprint" "pkorsako_footprint:R_0603"
 			(at 101.6 38.1 0)
 			(hide yes)
@@
 			)
 		)
-		(property "Footprint" ""
+		(property "Footprint" "pkorsako_footprint:SW_SPST_B3U-1000P"
 			(at 153.67 53.34 0)
 			(hide yes)
@@
 			)
 		)
-		(property "Footprint" ""
+		(property "Footprint" "pkorsako_footprint:TQFP-32_7x7_Pitch0.8mm"
 			(at 59.69 128.27 0)
 			(hide yes)
@@
 			)
 		)
-		(property "Footprint" ""
+		(property "Footprint" "pkorsako_footprint:R_0603"
 			(at 165.1 45.72 0)
 			(hide yes)
@@
 			)
 		)
-		(property "Footprint" ""
+		(property "Footprint" "pkorsako_footprint:Crystal_SMD_3225"
 			(at 99.06 121.92 0)
 			(hide yes)
@@
 			)
 		)
-		(property "Footprint" ""
+		(property "Footprint" "pkorsako_footprint:C_0603"
 			(at 139.7 53.34 0)
 			(hide yes)
@@
 			)
 		)
-		(property "Footprint" ""
+		(property "Footprint" "pkorsako_footprint:PinHeader_1x12_P2.54mm"
 			(at 149.86 138.43 0)
 			(hide yes)
@@
 			)
 		)
-		(property "Footprint" ""
+		(property "Footprint" "pkorsako_footprint:Led_0603"
 			(at 101.6 52.07 0)
 			(hide yes)
@@
 			)
 		)
-		(property "Footprint" ""
+		(property "Footprint" "pkorsako_footprint:PinHeader_1x06_P2.54mm"
 			(at 201.93 143.51 0)
 			(hide yes)
@@
 			)
 		)
-		(property "Footprint" ""
+		(property "Footprint" "pkorsako_footprint:Led_0603"
 			(at 60.96 41.91 0)
 			(hide yes)
@@
 			)
 		)
-		(property "Footprint" ""
+		(property "Footprint" "pkorsako_footprint:R_0603"
 			(at 60.96 52.07 0)
 			(hide yes)
@@
 			)
 		)
-		(property "Footprint" ""
+		(property "Footprint" "pkorsako_footprint:C_0603"
 			(at 43.18 40.64 0)
 			(hide yes)
@@
 			)
 		)
-		(property "Footprint" ""
+		(property "Footprint" "pkorsako_footprint:C_0603"
 			(at 27.94 40.64 0)
 			(hide yes)
@@
 			)
 		)
-		(property "Footprint" ""
+		(property "Footprint" "pkorsako_footprint:C_0603"
 			(at 38.1 99.06 0)
 			(hide yes)

Commit message: finished
Connections:
- no-connect marks 2 -> 4
Changed lines of the file:
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@@
+	)
+	(no_connect
+		(at 74.93 135.89)
+	)
+	(no_connect
+		(at 74.93 133.35)
 	)
 	(no_connect
